Commit message: made_few changes

File: hannahbot_description/urdf/hannahbot_ros2_control.xacro (robot description, xacro)
@@ -28,4 +28,11 @@
             <state_interface name="position"/>
         </joint>
+        <joint name="hori_arm_claw_joint">
+            <command_interface name="position">
+                <param name="min">-${PI/2}</param>
+                <param name="max">${PI/2}</param>
+            </command_interface>
+            <state_interface name="position"/>
+        </joint>
         <joint name="joint_4">
             <command_interface name="position">
